File: delay-pedal.kicad_sch (KiCad schematic)
At the start: 35 parts, among them J1 9V, J2 IN 6.35mm, J3 OUT 6.35mm, K1 5V_DPDT, Q1 2N2219, SW1 Footswitch_momentary, U1 LM7805_TO220, U3 TL072

Commit message: Add routed 300 ms delay pedal prototype and hardware documentation
Parts:
- removed C1: 47u 25V, symbol Device:C_Polarized_US
- removed C3: 47u 16V, symbol Device:C_Polarized_US
- removed C6: 100 nF, symbol Device:C
- removed J1: 9V, symbol Connector:Jack-DC
- removed J2: IN 6.35mm, symbol Connector_Audio:AudioJack2
- removed J3: OUT 6.35mm, symbol Connector_Audio:AudioJack2
- removed K1: 5V_DPDT, symbol Relay:Relay_DPDT
- removed Q1: 2N2219, Package_TO_SOT_THT:TO-39-3, symbol Transistor_BJT:2N2219
- removed RV1: 10k lin TIME, symbol Device:R_Potentiometer
- removed RV2: 10k lin FB, symbol Device:R_Potentiometer
- removed RV3: 10k lin MIX, symbol Device:R_Potentiometer
- removed SW1: Footswitch_momentary, symbol Switch:SW_Push
- removed U3: TL072, symbol Amplifier_Operational:TL072
- added C1: 47u 25V, Capacitor_THT:CP_Radial_D6.3mm_P2.50mm, symbol Device:C_Polarized
- added C15: 100u 16V, Capacitor_THT:CP_Radial_D6.3mm_P2.50mm, symbol Device:C_Polarized
- added C16, C17, C19, C20: 100n, Capacitor_THT:C_Disc_D3.0mm_W1.6mm_P2.50mm, symbol Device:C
- added C18: 10n, Capacitor_THT:C_Disc_D3.0mm_W1.6mm_P2.50mm, symbol Device:C
- added C3, C6: 47u 16V, Capacitor_THT:CP_Radial_D6.3mm_P2.50mm, symbol Device:C_Polarized
- added D3, D4: BAT85, Diode_THT:D_DO-35_SOD27_P7.62mm_Horizontal, symbol Device:D_Schottky
- added J1: 9V IN: 1=+ 2=GND, Connector_PinHeader_2.54mm:PinHeader_1x02_P2.54mm_Vertical, symbol Connector_Generic:Conn_01x02
- added J2: INPUT: 1=TIP 2=SLEEVE, Connector_PinHeader_2.54mm:PinHeader_1x02_P2.54mm_Vertical, symbol Connector_Generic:Conn_01x02
- added J3: OUTPUT: 1=TIP 2=SLEEVE, Connector_PinHeader_2.54mm:PinHeader_1x02_P2.54mm_Vertical, symbol Connector_Generic:Conn_01x02
- added J4: TIME B10k, Connector_PinHeader_2.54mm:PinHeader_1x03_P2.54mm_Vertical, symbol Connector_Generic:Conn_01x03
- added J5: FEEDBACK B10k, Connector_PinHeader_2.54mm:PinHeader_1x03_P2.54mm_Vertical, symbol Connector_Generic:Conn_01x03
- added J6: MIX B10k, Connector_PinHeader_2.54mm:PinHeader_1x03_P2.54mm_Vertical, symbol Connector_Generic:Conn_01x03
- added J7: MOMENTARY NO, Connector_PinHeader_2.54mm:PinHeader_1x02_P2.54mm_Vertical, symbol Connector_Generic:Conn_01x02
- added J8: LED: 1=A 2=K, Connector_PinHeader_2.54mm:PinHeader_1x02_P2.54mm_Vertical, symbol Connector_Generic:Conn_01x02
- added JP1: POWER LINK: remove for USB, Connector_PinHeader_2.54mm:PinHeader_1x02_P2.54mm_Vertical, symbol Connector_Generic:Conn_01x02
- added K1: G5V-2-H1 DC5, Relay_THT:Relay_DPDT_Omron_G5V-2, symbol Relay:G5V-2
- added Q1: 2N3904, Package_TO_SOT_THT:TO-92_Inline_Wide, symbol Transistor_BJT:2N3904
- added R10: 22, Resistor_THT:R_Axial_DIN0204_L3.6mm_D1.6mm_P7.62mm_Horizontal, symbol Device:R
- added R11, R13: 1M, Resistor_THT:R_Axial_DIN0204_L3.6mm_D1.6mm_P7.62mm_Horizontal, symbol Device:R
- added R12: 100, Resistor_THT:R_Axial_DIN0204_L3.6mm_D1.6mm_P7.62mm_Horizontal, symbol Device:R
- added R14, R15, R16, R17: 10k, Resistor_THT:R_Axial_DIN0204_L3.6mm_D1.6mm_P7.62mm_Horizontal, symbol Device:R
- added R18: 1k, Resistor_THT:R_Axial_DIN0204_L3.6mm_D1.6mm_P7.62mm_Horizontal, symbol Device:R
- added R8: 2k2, Resistor_THT:R_Axial_DIN0204_L3.6mm_D1.6mm_P7.62mm_Horizontal, symbol Device:R
- added R9: 100k, Resistor_THT:R_Axial_DIN0204_L3.6mm_D1.6mm_P7.62mm_Horizontal, symbol Device:R
- added U3: MCP6002-I/P, Package_DIP:DIP-8_W7.62mm_Socket, symbol Amplifier_Operational:MCP6002-xP
- added U4: 23LC1024-I/P, Package_DIP:DIP-8_W7.62mm_Socket, symbol Delay:23LC1024
- C10, C8, C9: value C -> 100n; footprint (none) -> Capacitor_THT:C_Disc_D3.0mm_W1.6mm_P2.50mm
- C11, C12, C7: value 100 nF -> 10n; footprint (none) -> Capacitor_THT:C_Disc_D3.0mm_W1.6mm_P2.50mm
- C13: value 100 nF -> 1u film; footprint (none) -> Capacitor_THT:C_Rect_L7.2mm_W3.5mm_P5.00mm
- C14, C4: value 100 nF -> 100n; footprint (none) -> Capacitor_THT:C_Disc_D3.0mm_W1.6mm_P2.50mm
- C2: value 100 nF -> 330n; footprint (none) -> Capacitor_THT:C_Disc_D3.0mm_W1.6mm_P2.50mm
- C5: value 100 nF -> 100n film; footprint (none) -> Capacitor_THT:C_Rect_L7.2mm_W2.5mm_P5.00mm
- R1: footprint (none) -> Resistor_THT:R_Axial_DIN0204_L3.6mm_D1.6mm_P7.62mm_Horizontal
- R2, R3: value 100k -> 10k; footprint (none) -> Resistor_THT:R_Axial_DIN0204_L3.6mm_D1.6mm_P7.62mm_Horizontal
- R4: value R -> 2k2; footprint (none) -> Resistor_THT:R_Axial_DIN0204_L3.6mm_D1.6mm_P7.62mm_Horizontal
- R5, R6: value 1k -> 2k2; footprint (none) -> Resistor_THT:R_Axial_DIN0204_L3.6mm_D1.6mm_P7.62mm_Horizontal
- R7: value R -> 1k; footprint (none) -> Resistor_THT:R_Axial_DIN0204_L3.6mm_D1.6mm_P7.62mm_Horizontal
Connections:
- net BUF_IN: now also C5.2, R1.1, U3.3 (+); no longer C5.1, R1.2
- net FOOT: now also J7.1 (Pin_1), R17.2
- net GND: now also C10.2, C2.2, C4.2, C7.2, C8.2, C9.2, C1.2, C15.2, C16.2, C17.2, C18.2, C19.2, C20.2, C3.2, C6.2, D4.2 (A), J1.2 (Pin_2), J2.2 (Pin_2), J3.2 (Pin_2), J4.1 (Pin_1), J5.1 (Pin_1), J6.1 (Pin_1), J7.2 (Pin_2), J8.2 (Pin_2), Q1.1 (E), R11.2, R13.2, R9.2, U3.4 (V-), U4.4 (VSS); no longer C10.1, C2.1, C4.1, C8.1, C9.1, R4.1
- net MIX: now also C10.1, J6.2 (Pin_2); no longer C10.2
- net TIME: now also C8.1, J4.2 (Pin_2); no longer C8.2
- net VB_2V5: now also R1.2, C19.1, C6.1; no longer R1.1
- net OUT_ISO: now reaches C13.1
- net OUT_ISO: now also R12.2
- net Q_BASE: now reaches R7.2
- net Q_BASE: now also Q1.2 (B), R9.1
- net 9V_IN: now reaches D1.2 (A)
- net 9V_IN: now also J1.1 (Pin_1)
- net FX_OUT: now reaches C13.2
- net FX_OUT: now also K1.9, R13.1
- net 5V_REG: now reaches D2.1 (K)
- net 5V_REG: now also C4.1, U1.3 (VO), C3.1, JP1.1 (Pin_1), K1.1
- net ADC_F1: now reaches C7.1
- net ADC_F1: now also R4.2, R8.1
- net LED_CTRL: now reaches A1.10 (D7)
- net LED_CTRL: now also R18.1
- net SRAM_CS: now reaches A1.13 (D10)
- net SRAM_CS: now also R14.2, U4.1 (~{CS})
- net SPI_MOSI: now reaches A1.14 (D11)
- net SPI_MOSI: now also U4.5 (SI)
- net SPI_MISO: now reaches A1.15 (D12)
- net SPI_MISO: now also U4.2 (SO)
- net SPI_SCK: now reaches A1.16 (D13)
- net SPI_SCK: now also U4.6 (SCK)
- removed net +5V: A1.27 (+5V), C4.2, D2.2 (A), R2.1, U1.3 (VO)
- net +9V renamed 9V_PROT
- net 9V_PROT: now also C2.1, C1.1; no longer C2.2
- removed net A0_NET: A1.19 (A0), C7.2, R4.2
- net F1 renamed PWM_F1
- net FB renamed FEEDBACK
- net FEEDBACK: now also C9.1, J5.2 (Pin_2); no longer C9.2
- net PWM_FIL renamed PWM_FILTER
- net PWM_FILTER: now also U3.5 (+)
- net RELAY renamed RELAY_CTRL
- new net 5V_ANALOG: C15.1, C16.1, R10.2, R2.1, U3.8 (V+)
- new net 5V_LOGIC: A1.27 (+5V), C17.1, C20.1, D3.1 (K), J4.3 (Pin_3), J5.3 (Pin_3), J6.3 (Pin_3), JP1.2 (Pin_2), R10.1, R14.1, R15.1, R16.1, R17.1, U4.8 (VCC)
- new net AUDIO_ADC: A1.19 (A0), C18.1, D3.2 (A), D4.1 (K), R8.2
- new net BUF_OUT: R4.1, U3.1, U3.2 (-)
- new net BYPASS: K1.11, K1.6
- new net COIL_LOW: D2.2 (A), K1.16, Q1.3 (C)
- new net FX_IN: C5.1, K1.8
- new net INPUT: J2.1 (Pin_1), K1.4, R11.1
- new net LED_ANODE: J8.1 (Pin_1), R18.2
- new net OUTPUT: J3.1 (Pin_1), K1.13
- new net OUT_BUFFER: R12.1, U3.6 (-), U3.7
- new net SRAM_AUX: R15.2, U4.3 (SIO2)
- new net SRAM_HOLD: R16.2, U4.7 (~{HOLD})
- no-connect marks 21 -> 15
Other:
- note added: "16 ksample/s / 8-bit PWM; external SPI SRAM. Firmware and bench validation required."
- note added: "AUDIO INPUT / TRUE BYPASS | relay off = bypass"
- note added: "Audio filters are passive two-stage RC ladders (2k2 / 10n), about 2.7 kHz combined -3 dB."
- note added: "BIAS AND OUTPUT | both MCP6002 stages run from filtered 5 V"
- note added: "CONTROLS | three external B10k pots: 1=CCW/GND, 2=wiper, 3=CW/+5V"
- note added: "Default-off pull-down R9; D2 cathode (band) to +5V_REG. Do not substitute a different relay pinout."
- note added: "Fit JP1 for normal 9 V operation. Remove JP1 BEFORE connecting USB. Relay uses 5V_REG."
- note added: "NANO / EXTERNAL MEMORY | 4,800 sample bytes for 300 ms at 16 ksample/s"
- note added: "NANO DELAY | 300 ms TARGET | PROTOTYPE REV A"
- note added: "POWER | regulated 9 V adapter; wire the external jack to J1"
- note added: "Prototype target: lo-fi mono delay. Timer/PWM/ADC scheduling, mix and feedback are implemented in firmware."
- note added: "RELAY DRIVER | use the H1 sensitivity version, 5 V coil"
- title: (none) -> Arduino Nano delay - 300 ms prototype

Commit message: Improve revision C PCB layout, labels and manufacturing documentation
Parts:
- A1: footprint Module:Arduino_Nano -> Delay:Arduino_Nano_EdgeUSB
Other:
- note added: "NANO DELAY | 300 ms TARGET | PROTOTYPE REV C"
- note removed: "NANO DELAY | 300 ms TARGET | PROTOTYPE REV A"
